File: bitaxeGamma.kicad_sch (KiCad schematic)
At the start: 20 parts, among them J1 54-00164

Commit message: Finish retouches and prepare manufacturing files
Parts:
- J1: MF (none) -> Tensility; MPN (none) -> 54-00164; PARTNO 54-00164 -> (none)
