File: bm1370.kicad_sch (KiCad schematic)
At the start: 47 parts, among them U5 MCP1824T-1202E/OT, U6 MCP1824T-0802E, U7 25MHz, U8 BM1370_mode1, U9 SN74AVC4T774

Commit message: Finish retouches and prepare manufacturing files
Parts:
- C26, C27, C28, C30, C31, C32, C33, C34, C35, C36, C41, C42, C44, C45, C46, C48: MF (none) -> Taiyo Yuden; MPN (none) -> EMK105BJ105MV-F; PARTNO EMK105BJ105MV-F -> (none)
- C29, C47, C49: MF (none) -> Samsung; MPN (none) -> CL05A104KO5NNNC; PARTNO CL05A104KO5NNNC -> (none)
- C43, C54: MF (none) -> Samsung; MPN (none) -> CL31A107MQHNNNE; PARTNO CL31A107MQHNNNE -> (none)
- R17, R26: MF (none) -> Yageo; MPN (none) -> RC0402FR-0710KL; PARTNO RC0402JR-0710KL -> (none)
- R18: MPN (none) -> RC0402FR-071KL; PARTNO RC0402FR-071KL -> (none)
- R19: MF (none) -> Yageo; MPN (none) -> RC0402FR-071KL; PARTNO RC0402FR-071KL -> (none)
- R20: MF (none) -> Yageo; MPN (none) -> RC0402FR-071KL; PARTNO RC0402FR-072KL -> (none)
- R21: MF (none) -> Yageo; MPN (none) -> RC0402FR-072KL; PARTNO RC0402FR-072KL -> (none)
- U5: MF (none) -> Microchip; MPN (none) -> MCP1824T-1202E/OT; PARTNO MCP1824T-1202E/OT -> (none)
- U6: MF (none) -> Microchip; MPN (none) -> MCP1824T-0802E/OT; PARTNO MCP1824T-0802E/OT -> (none)
- U7: Alt. MPN (none) -> OXLTDLJANF-25.000000; DK 5852-SX3M25.000E20F30THNTR-ND -> 1664-OXLTDLJANF-25.000000CT-ND; MF (none) -> SCTF; MPN (none) -> SX3M25.000E20F30THN; PARTNO SX3M25.000E20F30THN -> (none)
- U9: MF (none) -> TI; MPN (none) -> SN74AVC4T774PWR; PARTNO SN74AVC4T774PWR -> (none)
