File: esp32.kicad_sch (KiCad schematic)
At the start: 24 parts, among them J2 TC2030-IDC, J3 Conn_01x04, J4 Conn_01x06, J5 USB_C_Receptacle_USB2.0, SW1 GT-TC029B-H025-L1N, SW2 GT-TC029B-H025-L1N, U3 RT9080-33GJ5, U4 ESP32-S3-WROOM-1

Commit message: Finish retouches and prepare manufacturing files
Parts:
- C21, C22, C23: MF (none) -> Taiyo Yuden; MPN (none) -> EMK105BJ105MV-F; PARTNO EMK105BJ105MV-F -> (none)
- C6: MF (none) -> Murata; MPN (none) -> GRM188R61E106KA73D; PARTNO GRM188R61E106KA73D -> (none)
- J5: MF (none) -> GCT; MPN (none) -> USB4105-GF-A; PARTNO USB4105-GF-A -> (none)
- R16: MF (none) -> Yageo; MPN (none) -> RC0402FR-0710KL; PARTNO RC0402JR-0710KL -> (none)
- R27, R28: MF (none) -> Yageo; MPN (none) -> RC0402FR-135K6L; PARTNO RC0402FR-135K6L -> (none)
- R29, R30: DK RMCF0402JT5K10CT-ND -> 311-5.10KLRCT-ND; LCSC (none) -> C25905; LCSC Part C25905 -> (none); MF (none) -> Yageo; MPN (none) -> RC0402FR-075K1L; PARTNO RMCF0402JT5K10 -> (none)
- SW1, SW2: MF (none) -> CIT; MPN (none) -> CS1213AGF260; PARTNO CS1213AGF260 -> (none)
- U3: MF (none) -> Richtek; MPN (none) -> RT9080-33GJ5; PARTNO RT9080-33GJ5 -> (none)
- U4: MF (none) -> Espressif; MPN (none) -> ESP32-S3-WROOM-1-N16R8; PARTNO ESP32-S3-WROOM-1-N16R8 -> (none)
