File: fan.kicad_sch (KiCad schematic)
At the start: 14 parts, among them J6 Conn_01x04, U10 EMC2101

Commit message: Finish retouches and prepare manufacturing files
Parts:
- C50: MF (none) -> Samsung; MPN (none) -> CL05B471KB5NNNC; PARTNO CL05B471KB5NNNC -> (none)
- C51: MF (none) -> Samsung; MPN (none) -> CL31A107MQHNNNE; PARTNO CL31A107MQHNNNE -> (none)
- C52, C53: MF (none) -> Samsung; MPN (none) -> CL05A104KO5NNNC; PARTNO CL05A104KO5NNNC -> (none)
- J6: MF (none) -> Molex; MPN (none) -> 0470531000; PARTNO 0470531000 -> (none)
- R22, R23: MF (none) -> Yageo; MPN (none) -> RC0402FR-07100RL; PARTNO RC0402FR-07100RL -> (none)
- R24: MF (none) -> Yageo; MPN (none) -> RC0402FR-135K6L; PARTNO RC0402FR-135K6L -> (none)
- R25: MF (none) -> Yageo; MPN (none) -> RC0402FR-0710KL; PARTNO RC0402JR-0710KL -> (none)
- U10: MF (none) -> Microchip; MPN (none) -> EMC2101-R-ACZL-TR; PARTNO EMC2101-R-ACZL-TR -> (none)
