File: power.kicad_sch (KiCad schematic)
At the start: 35 parts, among them T1 net-tie, U2 TPS546D24ARVFR

Commit message: Finish retouches and prepare manufacturing files
Parts:
- C1, C5: MF (none) -> Taiyo Yuden; MPN (none) -> EMK105BJ105MV-F; PARTNO EMK105BJ105MV-F -> (none)
- C11: MF (none) -> Yageo; MPN (none) -> CC0805KRX7R9BB102; PARTNO CC0805KRX7R9BB102 -> (none)
- C12, C8: MF (none) -> Samsung; MPN (none) -> CL05A104KO5NNNC; PARTNO CL05A104KO5NNNC -> (none)
- C13: MF (none) -> WE; MPN (none) -> 885012005013; PARTNO 885012005013 -> (none)
- C17, C18, C19, C2, C20, C3, C4: MF (none) -> Samsung; MPN (none) -> CL31A107MQHNNNE; PARTNO CL31A107MQHNNNE -> (none)
- C7, C9: MF (none) -> Murata; MPN (none) -> GRM188R61E106KA73D; PARTNO GRM188R61E106KA73D -> (none)
- L1: Alt. MPN (none) -> 104CDMCCDS-R30MC; DK (none) -> 732-3024-1-ND; MF (none) -> WE; MPN (none) -> 744308033; PARTNO 104CDMCCDS-R30MC -> (none)
- R1: MF (none) -> Yageo; MPN (none) -> RC0402FR-078K25L; PARTNO RC0402FR-078K25L -> (none)
- R10: MF (none) -> Yageo; MPN (none) -> RC0402FR-0768K1L; PARTNO RC0402FR-0768K1L -> (none)
- R11: MF (none) -> Yageo; MPN (none) -> RC0402FR-0710RL; PARTNO RC0402FR-0710RL -> (none)
- R12: MF (none) -> Stackpole; MPN (none) -> CSR1206FT1R00; PARTNO CSR1206FT1R00 -> (none)
- R13, R14: MF (none) -> Yageo; MPN (none) -> RC0402FR-0749R9L; PARTNO RC0402FR-0749R9L -> (none)
- R15: MF (none) -> Yageo; MPN (none) -> RC0402FR-0710KL; PARTNO RC0402JR-0710KL -> (none)
- R5: MF (none) -> Yageo; MPN (none) -> RC0402FR-0714K7L; PARTNO RC0402FR-0714K7L -> (none)
- R6: MF (none) -> Yageo; MPN (none) -> RC0402FR-070RL; PARTNO RC0402JR-070RL -> (none)
- R8: MF (none) -> Yageo; MPN (none) -> RC0402FR-073K74L; PARTNO RC0402FR-073K74L -> (none)
- R9: MF (none) -> Yageo; MPN (none) -> RC0402FR-0711K8L; PARTNO RC0402FR-0711K8L -> (none)
- T1: MPN (none) -> 2R5TPE220MAFB; PARTNO 2R5TPE220MAFB -> (none)
- U2: MF (none) -> TI; MPN (none) -> TPS546D24ARVFR; PARTNO TPS546D24ARVFR -> (none)
